File: src/transformation/nand2.sch (EAGLE design)
At the start: 7 parts, among them Q1 BSS92, Q2 BSS92, Q3 BSS97, Q4 BSS97

Commit message: added a slightly changed .sch file for comparing two eagle models afterwards
Parts:
- added Q5: BSS92, transistor-fet:BSS92
Changed lines of the file:
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@@
 <part name="A" library="pinhead" deviceset="PINHD-1X1" device=""/>
 <part name="B" library="pinhead" deviceset="PINHD-1X1" device=""/>
+<part name="Q5" library="transistor-fet" deviceset="BSS92" device="">
+<attribute name="P1" value="0001"/>
+<attribute name="TEST2" value="5"/>
+</part>
 </parts>
 <sheets>
@@
 <instance part="A" gate="G$1" x="-215.9" y="137.16" rot="R180"/>
 <instance part="B" gate="G$1" x="-215.9" y="119.38" rot="R180"/>
+<instance part="Q5" gate="G$1" x="-213.36" y="185.42">
+<attribute name="P1" x="-213.36" y="185.42" size="1.778" layer="96" display="off"/>
+<attribute name="TEST2" x="-213.36" y="185.42" size="1.778" layer="96" display="off"/>
+</instance>
 </instances>
 <busses>
