File: src/transformation/nand.sch (EAGLE design)
At the start: 7 parts, among them Q1 BSS92, Q2 BSS92, Q3 BSS97, Q4 BSS97

Commit message: completed transformation from eaglemodel to a .sch file
Parts:
- Q1: UID (none) -> 8
